File: Adafruit ESP8266 Feather.sch (EAGLE design)
At the start: 35 parts, among them IC1 CP2104, Q1 mmbt2222, Q2 mmbt2222, SW2 KMR2, U2 SPX3819, U3 MCP73831T-2ACI/OT, X1 JSTPH, X2 ESP-12, X4 20329

Commit message: added low cost version
Parts:
- removed C2: 10uF, microbuilder:CAP_CERAMIC0805-NOOUTLINE
- removed C3: 10µF, microbuilder:CAP_CERAMIC0805-NOOUTLINE
- removed CHG: ORANGE, microbuilder:LED0805_NOOUTLINE
- removed D3: RED, microbuilder:LED0805_NOOUTLINE
- removed IC1: CP2104, microbuilder:CP2104
- removed R10, R2: 1K, microbuilder:RESISTOR_0603_NOOUT
- removed R8: 10K\, microbuilder:RESISTOR_0603_NOOUT
- removed SJ1: (no value), microbuilder:SOLDERJUMPER_CLOSED
- removed U3: MCP73831T-2ACI/OT, microbuilder:MCP73831/2
- removed X1: JSTPH, microbuilder:CON_JST_PH_2PIN
Connections:
- removed net N$1: CHG.C, R2.1
- removed net N$2: IC1G$1.D+, X4.D+
- removed net N$3: R2.2, U3.STAT
- removed net N$4: R8.1, U3.PROG
- removed net N$5: D3.C, R10.2
- removed net N$6: IC1G$1.D-, X4.D-
- removed net N$7: SJ1.1, U3.VBAT
- net 3.3V: no longer C2.1, D3.A, IC1G$1.REGIN, IC1G$1.VDD, IC1G$1.VIO
- net DTR: no longer IC1G$1.DTR
- net GND: no longer C2.2, C3.2, IC1G$1.GND, IC1G$2.TP, R8.2, U3.VSS, X1.1
- net GPIO0: no longer R10.1
- net RTS: no longer IC1G$1.RTS
- net TXD: no longer IC1G$1.RXD
- net USB_RX: no longer IC1G$1.TXD
- net VBAT: no longer C3.1, SJ1.2, X1.2
- net VBUS: no longer CHG.A, IC1G$1.VBUS, U3.VDD
Other:
- note removed: "1.0K = 1000mA"
- note removed: "10K = 100mA"
- note removed: "2.0K = 500mA"
- note removed: "5.0K = 200mA"
- note removed: "LED"
- note removed: "LIPO CHARGING"
- note removed: "USB TO SERIAL CONVERTER"

Commit message: through hole parts
Parts:
- removed Q1, Q2: mmbt2222, SparkFun:TRANSISTOR_NPNSOT23-3
- removed R1, R4, R7, R9: 10K, microbuilder:RESISTOR_0603_NOOUT
- removed R11: 1K, microbuilder:RESISTOR_0603MP
- removed R5: 10K, microbuilder:RESISTOR_0603MP
- removed R6: 4.7K, microbuilder:RESISTOR_0603_NOOUT
- removed SW2: KMR2, microbuilder:SWITCH_TACT_SMT4.6X2.8
- removed U$34, U$35: FIDUCIAL"", microbuilder:FIDUCIAL""
- removed U2: SPX3819, microbuilder:VREG_SOT23-5
- removed X4: 20329, microbuilder:USB_MICRO_20329_V2
- added IC2: LD117AV33, v-reg:LD117AV33
- added SW1: (no value), adafruit:SWITCH_PUSHBUTTONEVQ-PE
- C6, C8: device microbuilder:CAP_CERAMIC0805-NOOUTLINE -> rcl:C-EU025-024X044
- C7: device microbuilder:CAP_CERAMIC0603_NO -> rcl:C-EU025-024X044
- D4: device microbuilder:DIODE-SCHOTTKYSOD-123 -> adafruit:SCHOTTKY-DIODEDO41-7
- R3: device microbuilder:RESISTOR_0603_NOOUT -> rcl:R-EU_0204/5
Connections:
- removed net DTR: Q2.E, R4.1
- removed net N$12: Q1.B, R4.2
- removed net N$13: Q2.B, R5.2
- removed net RTS: Q1.E, R5.1
- removed net USB_RX: R11.1
- net 3.3V: now also IC2.OUT; no longer R1.2, R9.2, U2.OUT
- net CH_PD: no longer R1.1
- net EN: no longer R7.1, U2.EN
- net GND: now also IC2.ADJ, SW1.P$2; no longer R6.1, SW2.P, SW2.P1, U2.GND, X4.GND
- net GPIO0: no longer Q2.C
- net GPIO15: no longer R6.2
- net GPIO2: no longer R9.1
- net RESET: now also SW1.P$1; no longer Q1.C, SW2.S, SW2.S1
- net RXD: no longer R11.2
- net VBUS: now also IC2.IN; no longer R7.2, U2.IN, X4.VBUS
Other:
- moved on the sheet: C6, C7, C8
